File: tia.sch (KiCad schematic (older format))
At the start: 49 parts, among them P1 CONN_01X02, P101 CONN_01X02, P102 CONN_01X02, P103 CONN_01X02, P2 CONN_01X02, Q1 MMBT3904, Q2 MMBT3904, Q3 MMBT3904, Q4 MMBT3904, Q5 MMBT3904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

Commit message: schematic as PDF
Other:
- note added: "PCB layout by Lasse OH3HZB (2022), based on work by Jan OM2ATC.\nOriginal design by Wes Hayward W7ZOI and Bob Kopski K3NHI."
- note added: "Termination insensitive IF amplifier board (dual TIA)"
- moved on the sheet: C1, C10, C11, C2, C3, C4, C5, C6, C7, C8, C9, D1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
